File: Nano-Tek.kicad_pcb (KiCad board)
At the start: 4 copper layers, 55 x 42 mm, 48 parts, among them CN1 POWER_IN, CN2 USB, CN3 Floppy 34, J1 Sound, J2 USB_Prog, J3 OLED, J4 Encoder+SER, J5 GND, Q1 MMBT3904, U1 STM32F105RBT6, U2 74LCX07, U3 AP2112K-3.3, X1 8MHz

Commit message: Rev 1.1 with Rotated Floppy Header
Rotated floppy header for better fit in some motherboards like A4000D.
Parts:
- moved CN3 41.5 mm to (87.9, 54.1), turned to -90 degrees
- moved R6 23.6 mm to (75.8, 45.9), turned to 0 degrees
- moved R11 10.5 mm to (73.9, 49.3)
- moved R9 10.5 mm to (63.4, 49.3)
- moved R7 3.50 mm to (70.4, 49.3)
- moved R8 3.50 mm to (66.9, 49.3)
- moved J1 1.27 mm to (86.2, 44.4)
Routing:
- net _CHNG: track 15.7 -> 64.7 mm
- net _RDY: track 55.9 -> 17.7 mm
- net _DKRD: track 36.8 -> 8.60 mm
- net _SIDE: track 24.3 -> 48.4 mm
- net _INDEX: track 6.69 -> 29.5 mm, vias 1 -> 2
- net _TRK0: track 29.8 -> 8.10 mm
- net _WPROT: track 30.8 -> 18.9 mm
- net _DKWE: track 30.9 -> 19.1 mm, vias 1 -> 2
- net +5V: track 135.3 -> 127.4 mm
- net _SEL0: track 35.0 -> 27.1 mm, vias 1 -> 0
- net _STEP: track 26.1 -> 28.2 mm
- net DIR: track 29.4 -> 31.4 mm
- net SPK-: track 5.79 -> 7.70 mm
- net _DKWD: track 24.6 -> 25.7 mm
- net GND: vias 83 -> 82
Other:
- board text added: "ROTATED HEADER"
